File: Fuente.sch (KiCad schematic (older format))
At the start: 15 parts, among them IC1 LM2577HV-ADJ, J1 CONN_01X02, J8 CONN_01X02, U3 LM7805

Commit message: Primera version del PCB
Parts:
- removed U3: LM7805, symbol LM7805
- added U3: 7805, TO_SOT_Packages_THT:TO-220-3_Vertical, symbol 7805
- C1, C2, C3, C4, C5: footprint (none) -> Capacitors_ThroughHole:C_Disc_D3.0mm_W2.0mm_P2.50mm
- D1, D2: footprint (none) -> Diodes_ThroughHole:D_A-405_P7.62mm_Horizontal
- IC1: footprint (none) -> TO_SOT_Packages_THT:TO-220-5_Vertical
- J1: footprint (none) -> Connect:bornier2
- J8: footprint (none) -> Pin_Headers:Pin_Header_Straight_2x01_Pitch2.54mm
- L1: footprint (none) -> Choke_Toroid_ThroughHole:Choke_Toroid_horizontal_Diameter3-5mm_Amidon-T12
- R1, R2, R3: footprint (none) -> Resistors_ThroughHole:R_Axial_DIN0204_L3.6mm_D1.6mm_P5.08mm_Horizontal
Connections:
- net +12V: now also U3.VI
- net GND: now also U3.GND
- net at C5.1, J8.1 (P1): now also U3.VO
Changed lines of the file:
@@
 F 0 "IC1" H 5200 3900 40  0000 L BNN
 F 1 "LM2577HV-ADJ" H 5200 3200 40  0000 L TNN
-F 2 "" H 7300 3450 30  0000 C CIN
+F 2 "TO_SOT_Packages_THT:TO-220-5_Vertical" H 7300 3450 30  0001 C CIN
 F 3 "" H 7300 3450 60  0000 C CNN
 F 4 "LM2577T-ADJ/NOPB-ND" H 5700 3600 60  0001 C CNN "Digikey#"
@@
 F 0 "R3" V 7180 3900 50  0000 C CNN
 F 1 "2K" V 7100 3900 50  0000 C CNN
-F 2 "" V 7030 3900 50  0001 C CNN
+F 2 "Resistors_ThroughHole:R_Axial_DIN0204_L3.6mm_D1.6mm_P5.08mm_Horizontal" V 7030 3900 50  0001 C CNN
 F 3 "" H 7100 3900 50  0001 C CNN
 F 4 "S2KQTR-ND" H 7100 3900 60  0001 C CNN "Digikey#"
@@
 F 0 "R2" V 7180 3400 50  0000 C CNN
 F 1 "1K8" V 7100 3400 50  0000 C CNN
-F 2 "" V 7030 3400 50  0001 C CNN
+F 2 "Resistors_ThroughHole:R_Axial_DIN0204_L3.6mm_D1.6mm_P5.08mm_Horizontal" V 7030 3400 50  0001 C CNN
 F 3 "" H 7100 3400 50  0001 C CNN
 F 4 "S1.8KQTR-ND" H 7100 3400 60  0001 C CNN "Digikey#"
@@
 F 0 "L1" V 5650 3050 50  0000 C CNN
 F 1 "100u" V 5775 3050 50  0000 C CNN
-F 2 "" H 5700 3050 50  0001 C CNN
+F 2 "Choke_Toroid_ThroughHole:Choke_Toroid_horizontal_Diameter3-5mm_Amidon-T12" H 5700 3050 50  0001 C CNN
 F 3 "" H 5700 3050 50  0001 C CNN
 F 4 "M8354-ND" H 5700 3050 60  0001 C CNN "Digikey#"
@@
 F 0 "D2" H 6450 3150 50  0000 C CNN
 F 1 "1N5821" H 6450 2950 50  0000 C CNN
-F 2 "" H 6450 3050 50  0001 C CNN
+F 2 "Diodes_ThroughHole:D_A-405_P7.62mm_Horizontal" H 6450 3050 50  0001 C CNN
 F 3 "" H 6450 3050 50  0001 C CNN
 F 4 "1N5821FSCT-ND" H 6450 3050 60  0001 C CNN "Digikey#"
@@
 F 0 "C3" H 7525 3750 50  0000 L CNN
 F 1 "1000u" H 7525 3550 50  0000 L CNN
-F 2 "" H 7538 3500 50  0001 C CNN
+F 2 "Capacitors_ThroughHole:C_Disc_D3.0mm_W2.0mm_P2.50mm" H 7538 3500 50  0001 C CNN
 F 3 "" H 7500 3650 50  0001 C CNN
 F 4 "1189-1583-3-ND" H 7500 3650 60  0001 C CNN "Digikey#"
@@
 F 0 "R1" V 4680 3650 50  0000 C CNN
 F 1 "2K2" V 4600 3650 50  0000 C CNN
-F 2 "" V 4530 3650 50  0001 C CNN
+F 2 "Resistors_ThroughHole:R_Axial_DIN0204_L3.6mm_D1.6mm_P5.08mm_Horizontal" V 4530 3650 50  0001 C CNN
 F 3 "" H 4600 3650 50  0001 C CNN
 F 4 "S2.2KQTR-ND" H 4600 3650 60  0001 C CNN "Digikey#"
@@
 F 0 "C2" H 4375 4000 50  0000 L CNN
 F 1 "0,33u" H 4375 3800 50  0000 L CNN
-F 2 "" H 4388 3750 50  0001 C CNN
+F 2 "Capacitors_ThroughHole:C_Disc_D3.0mm_W2.0mm_P2.50mm" H 4388 3750 50  0001 C CNN
 F 3 "" H 4350 3900 50  0001 C CNN
 F 4 "493-10258-3-ND" H 4350 3900 60  0001 C CNN "Digikey#"
@@
 F 0 "C1" H 4075 3750 50  0000 L CNN
 F 1 "0,1u" H 4075 3550 50  0000 L CNN
-F 2 "" H 4088 3500 50  0001 C CNN
+F 2 "Capacitors_ThroughHole:C_Disc_D3.0mm_W2.0mm_P2.50mm" H 4088 3500 50  0001 C CNN
 F 3 "" H 4050 3650 50  0001 C CNN
 F 4 "493-10498-3-ND" H 4050 3650 60  0001 C CNN "Digikey#"
@@
 F 0 "J1" H 2200 3700 50  0000 C CNN
 F 1 "CONN_01X02" V 2300 3550 50  0000 C CNN
-F 2 "" H 2200 3550 50  0001 C CNN
+F 2 "Connect:bornier2" H 2200 3550 50  0001 C CNN
 F 3 "" H 2200 3550 50  0001 C CNN
 F 4 "277-1667-ND" H 2200 3550 60  0001 C CNN "Digikey#"
@@
 F 0 "D1" H 2600 3600 50  0000 C CNN
 F 1 "1N5821" H 2600 3400 50  0000 C CNN
-F 2 "" H 2600 3500 50  0001 C CNN
+F 2 "Diodes_ThroughHole:D_A-405_P7.62mm_Horizontal" H 2600 3500 50  0001 C CNN
 F 3 "" H 2600 3500 50  0001 C CNN
 F 4 "1N5821FSCT-ND" H 2600 3500 60  0001 C CNN "Digikey#"
@@
 $EndComp
 $Comp
-L LM7805 U3
-U 1 1 591267BB
-P 9350 3500
-F 0 "U3" H 9500 3304 50  0000 C CNN
-F 1 "LM7805" H 9350 3700 50  0000 C CNN
-F 2 "" H 9350 3500 50  0001 C CNN
-F 3 "" H 9350 3500 50  0001 C CNN
-F 4 "LM7805CT-ND" H 9350 3500 60  0001 C CNN "Digikey#"
-	1    9350 3500
-	1    0    0    -1
-$EndComp
-$Comp
 L GND #PWR028
 U 1 1 5912685A
@@
 F 0 "C4" H 8525 3800 50  0000 L CNN
 F 1 "0,33u" H 8525 3600 50  0000 L CNN
-F 2 "" H 8538 3550 50  0001 C CNN
+F 2 "Capacitors_ThroughHole:C_Disc_D3.0mm_W2.0mm_P2.50mm" H 8538 3550 50  0001 C CNN
 F 3 "" H 8500 3700 50  0001 C CNN
 F 4 "493-10258-3-ND" H 8500 3700 60  0001 C CNN "Digikey#"
@@
 F 0 "C5" H 9975 3800 50  0000 L CNN
 F 1 "0,1u" H 9975 3600 50  0000 L CNN
-F 2 "" H 9988 3550 50  0001 C CNN
+F 2 "Capacitors_ThroughHole:C_Disc_D3.0mm_W2.0mm_P2.50mm" H 9988 3550 50  0001 C CNN
 F 3 "" H 9950 3700 50  0001 C CNN
 F 4 "493-10498-3-ND" H 9950 3700 60  0001 C CNN "Digikey#"
@@
 F 0 "J8" H 10500 3800 50  0000 C CNN
 F 1 "CONN_01X02" V 10600 3650 50  0000 C CNN
-F 2 "" H 10500 3650 50  0001 C CNN
+F 2 "Pin_Headers:Pin_Header_Straight_2x01_Pitch2.54mm" H 10500 3650 50  0001 C CNN
 F 3 "" H 10500 3650 50  0001 C CNN
 F 4 "A1921-ND" H 10500 3650 60  0001 C CNN "Digikey#"
@@
 Wire Wire Line
 	9950 3450 9950 3550
+$Comp
+L 7805 U3
+U 1 1 59FF092A
+P 9350 3500
+F 0 "U3" H 9500 3304 50  0000 C CNN
+F 1 "7805" H 9350 3700 50  0000 C CNN
+F 2 "TO_SOT_Packages_THT:TO-220-3_Vertical" H 9350 3500 50  0001 C CNN
+F 3 "" H 9350 3500 50  0000 C CNN
+F 4 "LM7805CT-ND" H 9350 3500 60  0001 C CNN "Digikey#"
+F 5 "ON Semiconductor" H 9350 3500 60  0001 C CNN "Manf"
+F 6 "LM7805CT" H 9350 3500 60  0001 C CNN "Manf#"
+	1    9350 3500
+	1    0    0    -1
+$EndComp
 $EndSCHEMATC
